Commit message: move_arm.py works finally

File: src/piper_description/urdf/piper_description.urdf (robot description, URDF)
Before this commit: robot piper, 11 links, 10 joints
Links:
- removed link dummy_link
- added link world
- link base_link: geometry collision mesh filename=file:///home/mirage/Projects/posha_ws/src/piper_description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; visual mesh filename=file:///home/mirage/Projects/posha_ws/src/piper_description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
- link gripper_base: geometry collision mesh filename=file:///home/mirage/Projects/posha_ws/src/piper_description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; visual mesh filename=file:///home/mirage/Projects/posha_ws/src/piper_description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
- link link1: geometry collision mesh filename=file:///home/mirage/Projects/posha_ws/src/piper_description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; visual mesh filename=file:///home/mirage/Projects/posha_ws/src/piper_description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
- link link2: geometry collision mesh filename=file:///home/mirage/Projects/posha_ws/src/piper_description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; visual mesh filename=file:///home/mirage/Projects/posha_ws/src/piper_description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
- link link3: geometry collision mesh filename=file:///home/mirage/Projects/posha_ws/src/piper_description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; visual mesh filename=file:///home/mirage/Projects/posha_ws/src/piper_description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
- link link4: geometry collision mesh filename=file:///home/mirage/Projects/posha_ws/src/piper_description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; visual mesh filename=file:///home/mirage/Projects/posha_ws/src/piper_description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
- link link5: geometry collision mesh filename=file:///home/mirage/Projects/posha_ws/src/piper_description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; visual mesh filename=file:///home/mirage/Projects/posha_ws/src/piper_description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
- link link6: geometry collision mesh filename=file:///home/mirage/Projects/posha_ws/src/piper_description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; visual mesh filename=file:///home/mirage/Projects/posha_ws/src/piper_description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
- link link7: geometry collision mesh filename=file:///home/mirage/Projects/posha_ws/src/piper_description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; visual mesh filename=file:///home/mirage/Projects/posha_ws/src/piper_description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
- link link8: geometry collision mesh filename=file:///home/mirage/Projects/posha_ws/src/piper_description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; visual mesh filename=file:///home/mirage/Projects/posha_ws/src/piper_description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
Joints:
- removed joint base_to_dummy
- added joint world_to_base: type fixed, parent world, child base_link
